File: hardware/pcb-support/kicad/trimbox-support.sch (KiCad schematic (older format))
At the start: 19 parts, among them J1 RX / BEC, J2 GPS, U1 TPS563201, U2 LSM6DS3TR-C, U3 ESP32-S3 Mini Nano N16R8

Commit message: PCB support : J1 remplacé par deux picots servo coudés (J1 TX, J3 RX)
- Deux picots coudés 2,54 mm 1×3 (S, +, −) au bord gauche : deux rallonges
  servo ordinaires depuis les sorties 2 (TX → IO16) et 3 (RX ← IO15) du
  récepteur ; le + amène le BEC. À souder soi-même (hors BOM JLCPCB).
- GPS (J2, JST SH 4) remonté en haut à gauche ; trous de tenue des rangées 1-2
  gauche retirés ; C8 près de J2 ; routage refait.
- Contrôle : aucune erreur (isolement 0,17 mm), réseaux continus, KiCad et
  Gerber revérifiés ; pastilles traversantes carrées dessinées en carré.
- Schéma, sérigraphie (S / - / TX / RX), notice et visualiseur 2D/3D à jour.

Co-Authored-By: Claude Opus 5.5 <noreply@anthropic.com>
Claude-Session: https://claude.ai/code/session_012Z8LmxLPqA1DRecvv9zmWy
Parts:
- added R4: 4,7 kΩ, TrimBox:R_0402_1005Metric, symbol TrimBox:R
- C1: renamed from C2; value 100 nF 50 V -> 22 µF 25 V; footprint TrimBox:C_0603_1608Metric -> TrimBox:C_0805_2012Metric; LCSC C14663 -> C45783; MPN CC0603KRX7R9BB104 -> CL21A226MAQNNNE
- C2: renamed from C3; value 100 nF -> 100 nF 50 V; footprint TrimBox:C_0402_1005Metric -> TrimBox:C_0603_1608Metric; LCSC C1525 -> C14663; MPN CL05B104KO5NNNC -> CC0603KRX7R9BB104
- C3: renamed from R1; value 56 kΩ 1 % -> 100 nF; footprint TrimBox:R_0402_1005Metric -> TrimBox:C_0402_1005Metric; symbol TrimBox:R -> TrimBox:C; LCSC C25796 -> C1525; MPN 0402WGF5602TCE -> CL05B104KO5NNNC
- C5: renamed from D1; value B5819W -> 22 µF 25 V; footprint TrimBox:D_SOD-123 -> TrimBox:C_0805_2012Metric; symbol TrimBox:D_Schottky -> TrimBox:C; LCSC C8598 -> C45783; MPN B5819W -> CL21A226MAQNNNE
- C7: renamed from R3; value 4,7 kΩ -> 100 nF; footprint TrimBox:R_0402_1005Metric -> TrimBox:C_0402_1005Metric; symbol TrimBox:R -> TrimBox:C; LCSC C25900 -> C1525; MPN 0402WGF4701TCE -> CL05B104KO5NNNC
- C8: renamed from U2; value LSM6DS3TR-C -> 10 µF 25 V; footprint TrimBox:LGA-14_3x2.5mm_P0.5mm_LayoutBorder3x4y -> TrimBox:C_0805_2012Metric; symbol TrimBox:LSM6DS3TR-C -> TrimBox:C; LCSC C967633 -> C15850; MPN LSM6DS3TR-C -> CL21A106KAYNNNE
- D1: renamed from C8; value 10 µF 25 V -> B5819W; footprint TrimBox:C_0805_2012Metric -> TrimBox:D_SOD-123; symbol TrimBox:C -> TrimBox:D_Schottky; LCSC C15850 -> C8598; MPN CL21A106KAYNNNE -> B5819W
- J1: value RX / BEC -> Servo RX-TX; footprint TrimBox:JST_SH_SM05B-SRSS-TB_1x05-1MP_P1.00mm_Horizontal -> TrimBox:PinHeader_1x03_P2.54mm_Horizontal; symbol TrimBox:JST_SH_5 -> TrimBox:Servo_1x03; LCSC C136657 -> (none); MPN SM05B-SRSS-TB(LF)(SN) -> Picot coudé 1×3 2,54 mm
- J2: renamed from U1; value TPS563201 -> GPS; footprint TrimBox:SOT-23-6 -> TrimBox:JST_SH_SM04B-SRSS-TB_1x04-1MP_P1.00mm_Horizontal; symbol TrimBox:TPS563201 -> TrimBox:JST_SH_4; LCSC C116592 -> C160404; MPN TPS563201DDCR -> SM04B-SRSS-TB(LF)(SN)
- J3: renamed from J2; value GPS -> Servo RX-RX; footprint TrimBox:JST_SH_SM04B-SRSS-TB_1x04-1MP_P1.00mm_Horizontal -> TrimBox:PinHeader_1x03_P2.54mm_Horizontal; symbol TrimBox:JST_SH_4 -> TrimBox:Servo_1x03; LCSC C160404 -> (none); MPN SM04B-SRSS-TB(LF)(SN) -> Picot coudé 1×3 2,54 mm
- L1: renamed from C1; value 22 µF 25 V -> 3,3 µH; footprint TrimBox:C_0805_2012Metric -> TrimBox:L_Taiyo-Yuden_NR-30xx; symbol TrimBox:C -> TrimBox:L; LCSC C45783 -> C167749; MPN CL21A226MAQNNNE -> FNR3015S3R3MT
- R1: renamed from R2; value 10 kΩ 1 % -> 56 kΩ 1 %; LCSC C25744 -> C25796; MPN 0402WGF1002TCE -> 0402WGF5602TCE
- R2: renamed from C4; value 22 µF 25 V -> 10 kΩ 1 %; footprint TrimBox:C_0805_2012Metric -> TrimBox:R_0402_1005Metric; symbol TrimBox:C -> TrimBox:R; LCSC C45783 -> C25744; MPN CL21A226MAQNNNE -> 0402WGF1002TCE
- U1: renamed from L1; value 3,3 µH -> TPS563201; footprint TrimBox:L_Taiyo-Yuden_NR-30xx -> TrimBox:SOT-23-6; symbol TrimBox:L -> TrimBox:TPS563201; LCSC C167749 -> C116592; MPN FNR3015S3R3MT -> TPS563201DDCR
- U2: renamed from C6; value 100 nF -> LSM6DS3TR-C; footprint TrimBox:C_0402_1005Metric -> TrimBox:LGA-14_3x2.5mm_P0.5mm_LayoutBorder3x4y; symbol TrimBox:C -> TrimBox:LSM6DS3TR-C; LCSC C1525 -> C967633; MPN CL05B104KO5NNNC -> LSM6DS3TR-C
- renumbered C5 to C4, C7 to C6, R4 to R3
Connections:
- net +3V3: now also C6.2, U2.12 (CS), U2.5 (VDDIO), U2.8 (VDD), R4.1; no longer C6.1, C8.12 (CS), C8.5 (VDDIO), C8.8 (VDD), U2.2
- net +5V: now also C8.1, J2.2; no longer C5.1 (K), J3.2
- net BST: now also C3.2, U1.6 (VBST); no longer C2.2, J2.6 (VBST)
- net ELRS_RX: now also J3.1 (S); no longer J1.3
- net ELRS_TX: now also J1.1 (S); no longer J1.4
- net FB: now also R1.1, R2.2, U1.4 (VFB); no longer C3.1, J2.4 (VFB), R1.2
- net GND: now also C2.1, C4.1, C5.2, C6.1, C7.2, J1.3 (-), J2.MP, J3.3 (-), U1.1 (GND), U2.2 (SDx), U2.3 (SCx), U2.6 (GND), U2.7 (GND); no longer C4.2, C6.2, C8.1 (SDO/SA0), C8.3 (SCx), C8.6 (GND), C8.7 (GND), D1.2, J1.1, J1.5, J1.MP, J3.1, J3.MP, L1.1, R1.1
- net GPS_RX: now also J2.4; no longer J3.4
- net GPS_TX: now also J2.3; no longer J3.3
- net IMU_INT1: now also U2.4 (INT1); no longer C8.4 (INT1)
- net SCL: now also U2.13 (SCL), R4.2; no longer C8.13 (SCL), R3.2
- net SDA: now also R3.2, U2.14 (SDA); no longer C7.2, C8.14 (SDA)
- net SW: now also C3.1, L1.2; no longer C2.1, J2.2 (SW)
- net V5_BUCK: now also C4.2, C5.1, D1.2 (A), L1.1, R1.2; no longer C3.2, C4.1, C5.2 (A), R2.2, U1.1
- net VBEC: now also C2.2, J3.2 (+), U1.3 (VIN), U1.5 (EN); no longer J2.3 (VIN), J2.5 (EN), L1.2
- no-connect marks 18 -> 14
Other:
- note added: "J1 / J3 : picots coudés pour rallonges servo (S, +, -) : J1 sortie 2 du récepteur (TX -> IO16), J3 sortie 3 (RX <- IO15), + = BEC."
- note removed: "J1 : 1 masse, 2 +BEC (6-8,4 V), 3 vers RX du récepteur (IO15), 4 depuis TX du récepteur (IO16), 5 masse."
- moved on the sheet: C1, C2, C4, C6, R1, R3
Changed lines of the file:
@@
 $EndComp
 $Comp
-L TrimBox:JST_SH_5 J1
+L TrimBox:Servo_1x03 J1
 U 1 1 5F000002
-P 1300 1700
-F 0 "J1" H 1300 1400 50  0000 C CNN
-F 1 "RX / BEC" H 1300 2300 50  0000 C CNN
-F 2 "TrimBox:JST_SH_SM05B-SRSS-TB_1x05-1MP_P1.00mm_Horizontal" H 1300 1700 50  0001 C CNN
-F 3 "" H 1300 1700 50  0001 C CNN
-F 4 "C136657" H 1300 1700 50  0001 C CNN "LCSC"
-F 5 "SM05B-SRSS-TB(LF)(SN)" H 1300 1700 50  0001 C CNN "MPN"
-	1    1300 1700
+P 1300 1500
+F 0 "J1" H 1300 1300 50  0000 C CNN
+F 1 "Servo RX-TX" H 1300 1700 50  0000 C CNN
+F 2 "TrimBox:PinHeader_1x03_P2.54mm_Horizontal" H 1300 1500 50  0001 C CNN
+F 3 "" H 1300 1500 50  0001 C CNN
+F 4 "Picot coudé 1×3 2,54 mm" H 1300 1500 50  0001 C CNN "MPN"
+	1    1300 1500
+	1    0    0    -1
+$EndComp
+$Comp
+L TrimBox:Servo_1x03 J3
+U 1 1 5F000003
+P 1300 2300
+F 0 "J3" H 1300 2100 50  0000 C CNN
+F 1 "Servo RX-RX" H 1300 2500 50  0000 C CNN
+F 2 "TrimBox:PinHeader_1x03_P2.54mm_Horizontal" H 1300 2300 50  0001 C CNN
+F 3 "" H 1300 2300 50  0001 C CNN
+F 4 "Picot coudé 1×3 2,54 mm" H 1300 2300 50  0001 C CNN "MPN"
+	1    1300 2300
 	1    0    0    -1
 $EndComp
 $Comp
 L TrimBox:JST_SH_4 J2
-U 1 1 5F000003
+U 1 1 5F000004
 P 1300 3300
 F 0 "J2" H 1300 3050 50  0000 C CNN
@@
 $Comp
 L TrimBox:TPS563201 U1
-U 1 1 5F000004
+U 1 1 5F000005
 P 4300 1800
 F 0 "U1" H 4300 1550 50  0000 C CNN
@@
 $Comp
 L TrimBox:L L1
-U 1 1 5F000005
+U 1 1 5F000006
 P 6000 1800
 F 0 "L1" H 6000 1700 50  0000 C CNN
@@
 $Comp
 L TrimBox:C C1
-U 1 1 5F000006
+U 1 1 5F000007
 P 3100 2400
 F 0 "C1" H 3100 2300 50  0000 C CNN
@@
 $Comp
 L TrimBox:C C2
-U 1 1 5F000007
+U 1 1 5F000008
 P 3100 2800
 F 0 "C2" H 3100 2700 50  0000 C CNN
@@
 $Comp
 L TrimBox:C C3
-U 1 1 5F000008
+U 1 1 5F000009
 P 5500 1350
 F 0 "C3" H 5500 1250 50  0000 C CNN
@@
 $Comp
 L TrimBox:R R1
-U 1 1 5F000009
+U 1 1 5F00000A
 P 6100 2450
 F 0 "R1" H 6100 2350 50  0000 C CNN
@@
 $Comp
 L TrimBox:R R2
-U 1 1 5F00000A
+U 1 1 5F00000B
 P 6100 2850
 F 0 "R2" H 6100 2750 50  0000 C CNN
@@
 $Comp
 L TrimBox:C C4
-U 1 1 5F00000B
+U 1 1 5F00000C
 P 7000 1450
 F 0 "C4" H 7000 1350 50  0000 C CNN
@@
 $Comp
 L TrimBox:C C5
-U 1 1 5F00000C
+U 1 1 5F00000D
 P 7000 1850
 F 0 "C5" H 7000 1750 50  0000 C CNN
@@
 $Comp
 L TrimBox:D_Schottky D1
-U 1 1 5F00000D
+U 1 1 5F00000E
 P 7300 2350
 F 0 "D1" H 7300 2250 50  0000 C CNN
@@
 $Comp
 L TrimBox:C C8
-U 1 1 5F00000E
+U 1 1 5F00000F
 P 7300 2850
 F 0 "C8" H 7300 2750 50  0000 C CNN
@@
 $Comp
 L TrimBox:LSM6DS3TR-C U2
-U 1 1 5F00000F
+U 1 1 5F000010
 P 4300 5300
 F 0 "U2" H 4300 4850 50  0000 C CNN
@@
 $Comp
 L TrimBox:C C6
-U 1 1 5F000010
+U 1 1 5F000011
 P 2800 4700
 F 0 "C6" H 2800 4600 50  0000 C CNN
@@
 $Comp
 L TrimBox:C C7
-U 1 1 5F000011
+U 1 1 5F000012
 P 2800 5100
 F 0 "C7" H 2800 5000 50  0000 C CNN
@@
 $Comp
 L TrimBox:R R3
-U 1 1 5F000012
+U 1 1 5F000013
 P 5800 4600
 F 0 "R3" H 5800 4500 50  0000 C CNN
@@
 $Comp
 L TrimBox:R R4
-U 1 1 5F000013
+U 1 1 5F000014
 P 5800 5000
 F 0 "R4" H 5800 4900 50  0000 C CNN
@@
 	9000 5400 8900 5400
 Wire Wire Line
+	1550 1400 1650 1400
+Wire Wire Line
 	1550 1500 1650 1500
 Wire Wire Line
 	1550 1600 1650 1600
 Wire Wire Line
-	1550 1700 1650 1700
-Wire Wire Line
-	1550 1800 1650 1800
-Wire Wire Line
-	1550 1900 1650 1900
-Wire Wire Line
-	1300 2200 1300 2300
+	1550 2200 1650 2200
+Wire Wire Line
+	1550 2300 1650 2300
+Wire Wire Line
+	1550 2400 1650 2400
 Wire Wire Line
 	1550 3150 1650 3150
@@
 Text Label 8900 5400 2    50   ~ 0
 +5V
+Text Label 1650 1400 0    50   ~ 0
+ELRS_TX
 Text Label 1650 1500 0    50   ~ 0
-GND
+VBEC
 Text Label 1650 1600 0    50   ~ 0
+GND
+Text Label 1650 2200 0    50   ~ 0
+ELRS_RX
+Text Label 1650 2300 0    50   ~ 0
 VBEC
-Text Label 1650 1700 0    50   ~ 0
-ELRS_RX
-Text Label 1650 1800 0    50   ~ 0
-ELRS_TX
-Text Label 1650 1900 0    50   ~ 0
-GND
-Text Label 1300 2300 3    50   ~ 0
+Text Label 1650 2400 0    50   ~ 0
 GND
 Text Label 1650 3150 0    50   ~ 0
@@
 NoConn ~ 10200 3600
 NoConn ~ 10200 3700
-NoConn ~ 10200 3800
-NoConn ~ 10200 3900
-NoConn ~ 10200 4000
-NoConn ~ 10200 4100
 NoConn ~ 4850 5300
 NoConn ~ 4850 5400
@@
 PCB support à la taille de la carte ESP32 : composants sur cette face, ESP32 de l'autre côté (picots 2,54 mm).
 Text Notes 700 7250 0    50   ~ 0
-J1 : 1 masse, 2 +BEC (6-8,4 V), 3 vers RX du récepteur (IO15), 4 depuis TX du récepteur (IO16), 5 masse.
+J1 / J3 : picots coudés pour rallonges servo (S, +, -) : J1 sortie 2 du récepteur (TX -> IO16), J3 sortie 3 (RX <- IO15), + = BEC.
 Text Notes 700 7400 0    50   ~ 0
 J2 : 1 masse, 2 +5 V, 3 depuis TX du GPS (IO18), 4 vers RX du GPS (IO17) — ordre G V T R du HGLRC M100 Mini.

Commit message: PCB support : pastilles à souder pour les fils du récepteur (plus rien ne dépasse)
- J1 : 4 pastilles traversantes (trou 1,1 mm, pas 3 mm) TX, RX, +, − au
  bord gauche, à la place des picots coudés (J3 supprimé) : fils de deux
  rallonges servo coupées, aucune excroissance hors du contour.
- Routage refait ; contrôle : aucune erreur (isolement 0,177 mm), réseaux
  continus, KiCad et Gerber revérifiés.
- Schéma, sérigraphie, notice et visualiseur 2D/3D à jour.

Co-Authored-By: Claude Opus 5.5 <noreply@anthropic.com>
Claude-Session: https://claude.ai/code/session_012Z8LmxLPqA1DRecvv9zmWy
Parts:
- removed R4: 4,7 kΩ, TrimBox:R_0402_1005Metric, symbol TrimBox:R
- C1: renamed from L1; value 3,3 µH -> 22 µF 25 V; footprint TrimBox:L_Taiyo-Yuden_NR-30xx -> TrimBox:C_0805_2012Metric; symbol TrimBox:L -> TrimBox:C; LCSC C167749 -> C45783; MPN FNR3015S3R3MT -> CL21A226MAQNNNE
- C2: renamed from C1; value 22 µF 25 V -> 100 nF 50 V; footprint TrimBox:C_0805_2012Metric -> TrimBox:C_0603_1608Metric; LCSC C45783 -> C14663; MPN CL21A226MAQNNNE -> CC0603KRX7R9BB104
- C3: renamed from C2; value 100 nF 50 V -> 100 nF; footprint TrimBox:C_0603_1608Metric -> TrimBox:C_0402_1005Metric; LCSC C14663 -> C1525; MPN CC0603KRX7R9BB104 -> CL05B104KO5NNNC
- C4: renamed from R2; value 10 kΩ 1 % -> 22 µF 25 V; footprint TrimBox:R_0402_1005Metric -> TrimBox:C_0805_2012Metric; symbol TrimBox:R -> TrimBox:C; LCSC C25744 -> C45783; MPN 0402WGF1002TCE -> CL21A226MAQNNNE
- C6: renamed from U2; value LSM6DS3TR-C -> 100 nF; footprint TrimBox:LGA-14_3x2.5mm_P0.5mm_LayoutBorder3x4y -> TrimBox:C_0402_1005Metric; symbol TrimBox:LSM6DS3TR-C -> TrimBox:C; LCSC C967633 -> C1525; MPN LSM6DS3TR-C -> CL05B104KO5NNNC
- C8: renamed from D1; value B5819W -> 10 µF 25 V; footprint TrimBox:D_SOD-123 -> TrimBox:C_0805_2012Metric; symbol TrimBox:D_Schottky -> TrimBox:C; LCSC C8598 -> C15850; MPN B5819W -> CL21A106KAYNNNE
- D1: renamed from C5; value 22 µF 25 V -> B5819W; footprint TrimBox:C_0805_2012Metric -> TrimBox:D_SOD-123; symbol TrimBox:C -> TrimBox:D_Schottky; LCSC C45783 -> C8598; MPN CL21A226MAQNNNE -> B5819W
- J1: value Servo RX-TX -> Fils récepteur; footprint TrimBox:PinHeader_1x03_P2.54mm_Horizontal -> TrimBox:TrimBox_Pastilles_fils_4x1.1mm; symbol TrimBox:Servo_1x03 -> TrimBox:Pastilles_fils_4; MPN Picot coudé 1×3 2,54 mm -> Pastilles à souder
- J2: renamed from J3; value Servo RX-RX -> GPS; footprint TrimBox:PinHeader_1x03_P2.54mm_Horizontal -> TrimBox:JST_SH_SM04B-SRSS-TB_1x04-1MP_P1.00mm_Horizontal; symbol TrimBox:Servo_1x03 -> TrimBox:JST_SH_4; LCSC (none) -> C160404; MPN Picot coudé 1×3 2,54 mm -> SM04B-SRSS-TB(LF)(SN)
- L1: renamed from U1; value TPS563201 -> 3,3 µH; footprint TrimBox:SOT-23-6 -> TrimBox:L_Taiyo-Yuden_NR-30xx; symbol TrimBox:TPS563201 -> TrimBox:L; LCSC C116592 -> C167749; MPN TPS563201DDCR -> FNR3015S3R3MT
- R1: renamed from C3; value 100 nF -> 56 kΩ 1 %; footprint TrimBox:C_0402_1005Metric -> TrimBox:R_0402_1005Metric; symbol TrimBox:C -> TrimBox:R; LCSC C1525 -> C25796; MPN CL05B104KO5NNNC -> 0402WGF5602TCE
- R2: renamed from R1; value 56 kΩ 1 % -> 10 kΩ 1 %; LCSC C25796 -> C25744; MPN 0402WGF5602TCE -> 0402WGF1002TCE
- R3: renamed from C7; value 100 nF -> 4,7 kΩ; footprint TrimBox:C_0402_1005Metric -> TrimBox:R_0402_1005Metric; symbol TrimBox:C -> TrimBox:R; LCSC C1525 -> C25900; MPN CL05B104KO5NNNC -> 0402WGF4701TCE
- U1: renamed from J2; value GPS -> TPS563201; footprint TrimBox:JST_SH_SM04B-SRSS-TB_1x04-1MP_P1.00mm_Horizontal -> TrimBox:SOT-23-6; symbol TrimBox:JST_SH_4 -> TrimBox:TPS563201; LCSC C160404 -> C116592; MPN SM04B-SRSS-TB(LF)(SN) -> TPS563201DDCR
- U2: renamed from C8; value 10 µF 25 V -> LSM6DS3TR-C; footprint TrimBox:C_0805_2012Metric -> TrimBox:LGA-14_3x2.5mm_P0.5mm_LayoutBorder3x4y; symbol TrimBox:C -> TrimBox:LSM6DS3TR-C; LCSC C15850 -> C967633; MPN CL21A106KAYNNNE -> LSM6DS3TR-C
- renumbered C4 to C5, C6 to C7, R3 to R4
Connections:
- net +3V3: now also C6.2, C7.1, U2.12 (CS), U2.5 (VDDIO), U2.8 (VDD); no longer C6.12 (CS), C6.5 (VDDIO), C6.8 (VDD), C7.2
- net +5V: now also D1.1 (K), J2.2; no longer U1.2, U2.1
- net BST: now also C3.2, U1.6 (VBST); no longer L1.6 (VBST), R1.2
- net ELRS_RX: now also J1.2 (RX); no longer J2.1 (S)
- net FB: now also R1.1, R2.2, U1.4 (VFB); no longer C4.2, L1.4 (VFB), R2.1
- net GND: now also C1.1, C5.2, C7.2, C8.2, J1.4 (-), J2.1, J2.MP, R2.1, U2.1 (SDO/SA0), U2.3 (SCx), U2.6 (GND), U2.7 (GND); no longer C3.1, C5.1, C6.2 (SDx), C6.3 (SCx), C6.6 (GND), C6.7 (GND), C7.1, D1.2, J1.3 (-), J2.3 (-), L1.1 (GND), R3.2, U1.MP
- net GPS_RX: now also J2.4; no longer U1.4
- net GPS_TX: now also J2.3; no longer U1.3
- net IMU_INT1: now also U2.4 (INT1); no longer C6.4 (INT1)
- net SCL: now also R4.2, U2.13 (SCL); no longer C6.13 (SCL)
- net SDA: now also R3.2, U2.14 (SDA); no longer C6.14 (SDA), R4.2
- net SW: now also C3.1, U1.2 (SW); no longer C1.2, R1.1
- net V5_BUCK: now also C4.2, C5.1, D1.2 (A), L1.1, R1.2; no longer C1.1, C5.2, C8.2 (A), D1.1, R2.2
- net VBEC: now also C1.2, J1.3 (+), U1.3 (VIN), U1.5 (EN); no longer C3.2, J1.2 (+), J2.2 (+), L1.3 (VIN), L1.5 (EN)
Other:
- note added: "J1 : pastilles à souder : TX (sortie 2 du récepteur -> IO16), RX (sortie 3 <- IO15), + BEC, masse."
- note removed: "J1 / J3 : picots coudés pour rallonges servo (S, +, -) : J1 sortie 2 du récepteur (TX -> IO16), J3 sortie 3 (RX <- IO15), + = BEC."
- moved on the sheet: C2, C3, C5, C7, R2, R4
Changed lines of the file:
@@
 $EndComp
 $Comp
-L TrimBox:Servo_1x03 J1
+L TrimBox:Pastilles_fils_4 J1
 U 1 1 5F000002
-P 1300 1500
-F 0 "J1" H 1300 1300 50  0000 C CNN
-F 1 "Servo RX-TX" H 1300 1700 50  0000 C CNN
-F 2 "TrimBox:PinHeader_1x03_P2.54mm_Horizontal" H 1300 1500 50  0001 C CNN
-F 3 "" H 1300 1500 50  0001 C CNN
-F 4 "Picot coudé 1×3 2,54 mm" H 1300 1500 50  0001 C CNN "MPN"
-	1    1300 1500
-	1    0    0    -1
-$EndComp
-$Comp
-L TrimBox:Servo_1x03 J3
+P 1300 1900
+F 0 "J1" H 1300 1650 50  0000 C CNN
+F 1 "Fils récepteur" H 1300 2150 50  0000 C CNN
+F 2 "TrimBox:TrimBox_Pastilles_fils_4x1.1mm" H 1300 1900 50  0001 C CNN
+F 3 "" H 1300 1900 50  0001 C CNN
+F 4 "Pastilles à souder" H 1300 1900 50  0001 C CNN "MPN"
+	1    1300 1900
+	1    0    0    -1
+$EndComp
+$Comp
+L TrimBox:JST_SH_4 J2
 U 1 1 5F000003
-P 1300 2300
-F 0 "J3" H 1300 2100 50  0000 C CNN
-F 1 "Servo RX-RX" H 1300 2500 50  0000 C CNN
-F 2 "TrimBox:PinHeader_1x03_P2.54mm_Horizontal" H 1300 2300 50  0001 C CNN
-F 3 "" H 1300 2300 50  0001 C CNN
-F 4 "Picot coudé 1×3 2,54 mm" H 1300 2300 50  0001 C CNN "MPN"
-	1    1300 2300
-	1    0    0    -1
-$EndComp
-$Comp
-L TrimBox:JST_SH_4 J2
-U 1 1 5F000004
 P 1300 3300
 F 0 "J2" H 1300 3050 50  0000 C CNN
@@
 $Comp
 L TrimBox:TPS563201 U1
-U 1 1 5F000005
+U 1 1 5F000004
 P 4300 1800
 F 0 "U1" H 4300 1550 50  0000 C CNN
@@
 $Comp
 L TrimBox:L L1
-U 1 1 5F000006
+U 1 1 5F000005
 P 6000 1800
 F 0 "L1" H 6000 1700 50  0000 C CNN
@@
 $Comp
 L TrimBox:C C1
-U 1 1 5F000007
+U 1 1 5F000006
 P 3100 2400
 F 0 "C1" H 3100 2300 50  0000 C CNN
@@
 $Comp
 L TrimBox:C C2
-U 1 1 5F000008
+U 1 1 5F000007
 P 3100 2800
 F 0 "C2" H 3100 2700 50  0000 C CNN
@@
 $Comp
 L TrimBox:C C3
-U 1 1 5F000009
+U 1 1 5F000008
 P 5500 1350
 F 0 "C3" H 5500 1250 50  0000 C CNN
@@
 $Comp
 L TrimBox:R R1
-U 1 1 5F00000A
+U 1 1 5F000009
 P 6100 2450
 F 0 "R1" H 6100 2350 50  0000 C CNN
@@
 $Comp
 L TrimBox:R R2
-U 1 1 5F00000B
+U 1 1 5F00000A
 P 6100 2850
 F 0 "R2" H 6100 2750 50  0000 C CNN
@@
 $Comp
 L TrimBox:C C4
-U 1 1 5F00000C
+U 1 1 5F00000B
 P 7000 1450
 F 0 "C4" H 7000 1350 50  0000 C CNN
@@
 $Comp
 L TrimBox:C C5
-U 1 1 5F00000D
+U 1 1 5F00000C
 P 7000 1850
 F 0 "C5" H 7000 1750 50  0000 C CNN
@@
 $Comp
 L TrimBox:D_Schottky D1
-U 1 1 5F00000E
+U 1 1 5F00000D
 P 7300 2350
 F 0 "D1" H 7300 2250 50  0000 C CNN
@@
 $Comp
 L TrimBox:C C8
-U 1 1 5F00000F
+U 1 1 5F00000E
 P 7300 2850
 F 0 "C8" H 7300 2750 50  0000 C CNN
@@
 $Comp
 L TrimBox:LSM6DS3TR-C U2
-U 1 1 5F000010
+U 1 1 5F00000F
 P 4300 5300
 F 0 "U2" H 4300 4850 50  0000 C CNN
@@
 $Comp
 L TrimBox:C C6
-U 1 1 5F000011
+U 1 1 5F000010
 P 2800 4700
 F 0 "C6" H 2800 4600 50  0000 C CNN
@@
 $Comp
 L TrimBox:C C7
-U 1 1 5F000012
+U 1 1 5F000011
 P 2800 5100
 F 0 "C7" H 2800 5000 50  0000 C CNN
@@
 $Comp
 L TrimBox:R R3
-U 1 1 5F000013
+U 1 1 5F000012
 P 5800 4600
 F 0 "R3" H 5800 4500 50  0000 C CNN
@@
 $Comp
 L TrimBox:R R4
-U 1 1 5F000014
+U 1 1 5F000013
 P 5800 5000
 F 0 "R4" H 5800 4900 50  0000 C CNN
@@
 	9000 5400 8900 5400
 Wire Wire Line
-	1550 1400 1650 1400
-Wire Wire Line
-	1550 1500 1650 1500
-Wire Wire Line
-	1550 1600 1650 1600
-Wire Wire Line
-	1550 2200 1650 2200
-Wire Wire Line
-	1550 2300 1650 2300
-Wire Wire Line
-	1550 2400 1650 2400
+	1550 1750 1650 1750
+Wire Wire Line
+	1550 1850 1650 1850
+Wire Wire Line
+	1550 1950 1650 1950
+Wire Wire Line
+	1550 2050 1650 2050
 Wire Wire Line
 	1550 3150 1650 3150
@@
 Text Label 8900 5400 2    50   ~ 0
 +5V
-Text Label 1650 1400 0    50   ~ 0
+Text Label 1650 1750 0    50   ~ 0
 ELRS_TX
-Text Label 1650 1500 0    50   ~ 0
+Text Label 1650 1850 0    50   ~ 0
+ELRS_RX
+Text Label 1650 1950 0    50   ~ 0
 VBEC
-Text Label 1650 1600 0    50   ~ 0
-GND
-Text Label 1650 2200 0    50   ~ 0
-ELRS_RX
-Text Label 1650 2300 0    50   ~ 0
-VBEC
-Text Label 1650 2400 0    50   ~ 0
+Text Label 1650 2050 0    50   ~ 0
 GND
 Text Label 1650 3150 0    50   ~ 0
@@
 PCB support à la taille de la carte ESP32 : composants sur cette face, ESP32 de l'autre côté (picots 2,54 mm).
 Text Notes 700 7250 0    50   ~ 0
-J1 / J3 : picots coudés pour rallonges servo (S, +, -) : J1 sortie 2 du récepteur (TX -> IO16), J3 sortie 3 (RX <- IO15), + = BEC.
+J1 : pastilles à souder : TX (sortie 2 du récepteur -> IO16), RX (sortie 3 <- IO15), + BEC, masse.
 Text Notes 700 7400 0    50   ~ 0
 J2 : 1 masse, 2 +5 V, 3 depuis TX du GPS (IO18), 4 vers RX du GPS (IO17) — ordre G V T R du HGLRC M100 Mini.

Commit message: PCB support : 2 picots de tenue en haut à gauche, connexions décalées vers le bas
- Trous de tenue rangée 1 gauche (IO3, IO1) rétablis : l'ESP32 est tenue
  aux deux bouts du côté gauche (rangées 1 et 11) et sur toute la droite.
- Connecteur GPS J2 et pastilles J1 descendus ; C8 suit J2 ; routage refait.
- Contrôle : aucune erreur, réseaux continus, KiCad et Gerber revérifiés.

Co-Authored-By: Claude Opus 5.5 <noreply@anthropic.com>
Claude-Session: https://claude.ai/code/session_012Z8LmxLPqA1DRecvv9zmWy
Connections:
- no-connect marks 14 -> 16
Changed lines of the file:
@@
 NoConn ~ 10200 3600
 NoConn ~ 10200 3700
+NoConn ~ 10200 3800
+NoConn ~ 10200 3900
 NoConn ~ 4850 5300
 NoConn ~ 4850 5400
